File: hardware_v3/pi-parport.sch (KiCad schematic (older format))
At the start: 14 parts, among them J1 CONN_01X02, J2 40HAT, J3 Conn_02x13_Odd_Even, U1 CAT24C32, U2 SN74LVC161284DLR

Commit message: hardware_v4: add bypass capacitors, reroute traces
Do not route trace under resistor R5.  Move U2 upward to facilitate
rerouting this trace without adding more vias.

Also make sure footprints between schematic and PCB are in sync.

Update BOM with new parts.

Hardware version needs to be bumped due to PCB changes.  Version numbers
in schematic and PCB source changed, new files will need to be generated
later.
Parts:
- added C1, C2: 100nF, Capacitor_SMD:C_0805_2012Metric_Pad1.15x1.40mm_HandSolder, symbol Device:C
- U1: footprint Package_SO:SO-8_3.9x4.9mm_P1.27mm -> Package_SO:SOIC-8_3.9x4.9mm_P1.27mm
Connections:
- wire segments 171 -> 175
Changed lines of the file:
@@
 Sheet 1 1
 Title "Raspberry Pi IEEE 1284 Parallel Port HAT"
-Date "2019-11-30"
-Rev "V.3"
+Date "2020-07-20"
+Rev "V.4"
 Comp "WorlickWerx"
 Comment1 ""
@@
 F 0 "U1" H 3400 6300 50  0000 C CNN
 F 1 "CAT24C32" H 2800 6300 50  0000 C CNN
-F 2 "Package_SO:SO-8_3.9x4.9mm_P1.27mm" H 3050 5950 50  0001 C CNN
+F 2 "Package_SO:SOIC-8_3.9x4.9mm_P1.27mm" H 3050 5950 50  0001 C CNN
 F 3 "https://www.onsemi.com/pub/Collateral/CAT24C32-D.PDF" H 3050 5950 50  0001 C CNN
 F 4 "CAT24C32WI-GT3CT-ND" H 3050 5950 50  0001 C CNN "Digi-Key_PN"
@@
 	6900 4600 6900 4750
 Connection ~ 6900 4600
-$Comp
-L power:PWR_FLAG #FLG01
-U 1 1 5E42D6B7
-P 1500 4150
-F 0 "#FLG01" H 1500 4225 50  0001 C CNN
-F 1 "PWR_FLAG" V 1500 4277 50  0000 L CNN
-F 2 "" H 1500 4150 50  0001 C CNN
-F 3 "~" H 1500 4150 50  0001 C CNN
-	1    1500 4150
-	0    -1   -1   0
-$EndComp
 Wire Wire Line
 	1500 4150 1500 4250
@@
 Text Notes 750  5850 0    60   ~ 0
 Install J1 jumper\nor R1 shunt to\ndefeat EEPROM\nwrite protect.
+$Comp
+L Device:C C2
+U 1 1 5F163F92
+P 4550 1200
+F 0 "C2" H 4665 1246 50  0000 L CNN
+F 1 "100nF" H 4665 1155 50  0000 L CNN
+F 2 "Capacitor_SMD:C_0805_2012Metric_Pad1.15x1.40mm_HandSolder" H 4588 1050 50  0001 C CNN
+F 3 "~" H 4550 1200 50  0001 C CNN
+F 4 "399-1177-1-ND" H 4550 1200 50  0001 C CNN "Digi-Key_PN"
+F 5 "C0805C104Z5VACTU" H 4550 1200 50  0001 C CNN "MPN"
+F 6 "KEMET" H 4550 1200 50  0001 C CNN "Manufacturer"
+F 7 "0805" H 4550 1200 50  0001 C CNN "Package"
+F 8 "100nF, 50V capacitor" H 4550 1200 50  0001 C CNN "Description"
+F 9 "Bypass" H 4550 1200 50  0001 C CNN "Notes"
+	1    4550 1200
+	1    0    0    -1
+$EndComp
+$Comp
+L power:PWR_FLAG #FLG01
+U 1 1 5E42D6B7
+P 1500 4150
+F 0 "#FLG01" H 1500 4225 50  0001 C CNN
+F 1 "PWR_FLAG" V 1500 4277 50  0000 L CNN
+F 2 "" H 1500 4150 50  0001 C CNN
+F 3 "~" H 1500 4150 50  0001 C CNN
+	1    1500 4150
+	0    -1   -1   0
+$EndComp
+$Comp
+L Device:C C1
+U 1 1 5F167F1F
+P 4300 5350
+F 0 "C1" H 4415 5396 50  0000 L CNN
+F 1 "100nF" H 4415 5305 50  0000 L CNN
+F 2 "Capacitor_SMD:C_0805_2012Metric_Pad1.15x1.40mm_HandSolder" H 4338 5200 50  0001 C CNN
+F 3 "~" H 4300 5350 50  0001 C CNN
+F 4 "399-1177-1-ND" H 4300 5350 50  0001 C CNN "Digi-Key_PN"
+F 5 "C0805C104Z5VACTU" H 4300 5350 50  0001 C CNN "MPN"
+F 6 "KEMET" H 4300 5350 50  0001 C CNN "Manufacturer"
+F 7 "0805" H 4300 5350 50  0001 C CNN "Package"
+F 8 "100nF, 50V capacitor" H 4300 5350 50  0001 C CNN "Description"
+F 9 "Bypass" H 4300 5350 50  0001 C CNN "Notes"
+	1    4300 5350
+	1    0    0    -1
+$EndComp
+$Comp
+L power:+3.3V #PWR015
+U 1 1 5F177CFF
+P 4550 950
+F 0 "#PWR015" H 4550 800 50  0001 C CNN
+F 1 "+3.3V" H 4565 1123 50  0000 C CNN
+F 2 "" H 4550 950 50  0001 C CNN
+F 3 "" H 4550 950 50  0001 C CNN
+	1    4550 950
+	1    0    0    -1
+$EndComp
+Wire Wire Line
+	4550 950  4550 1050
+$Comp
+L power:GND #PWR016
+U 1 1 5F194F1A
+P 4550 1450
+F 0 "#PWR016" H 4550 1200 50  0001 C CNN
+F 1 "GND" H 4555 1277 50  0000 C CNN
+F 2 "" H 4550 1450 50  0001 C CNN
+F 3 "" H 4550 1450 50  0001 C CNN
+	1    4550 1450
+	1    0    0    -1
+$EndComp
+Wire Wire Line
+	4550 1350 4550 1450
+$Comp
+L power:+3.3V #PWR04
+U 1 1 5F1BDBF0
+P 4300 5100
+F 0 "#PWR04" H 4300 4950 50  0001 C CNN
+F 1 "+3.3V" H 4315 5273 50  0000 C CNN
+F 2 "" H 4300 5100 50  0001 C CNN
+F 3 "" H 4300 5100 50  0001 C CNN
+	1    4300 5100
+	1    0    0    -1
+$EndComp
+$Comp
+L power:GND #PWR05
+U 1 1 5F1BE58B
+P 4300 5600
+F 0 "#PWR05" H 4300 5350 50  0001 C CNN
+F 1 "GND" H 4305 5427 50  0000 C CNN
+F 2 "" H 4300 5600 50  0001 C CNN
+F 3 "" H 4300 5600 50  0001 C CNN
+	1    4300 5600
+	1    0    0    -1
+$EndComp
+Wire Wire Line
+	4300 5100 4300 5200
+Wire Wire Line
+	4300 5500 4300 5600
 $EndSCHEMATC
